File: KiCad Files/MainPCB/ENV_KB.kicad_pcb (KiCad board)
At the start: 2 copper layers, 347 x 156.3 mm, 231 parts

Commit message: test reroute, row 1
Parts:
- removed the H4 at (379.6, 193.4)
- removed the kibuzzard-628ADF99 at (334.4, 172.4)
- removed the kibuzzard-628AE061 at (356.2, 168.2)
- moved D78 374.2 mm to (404.1, 187.7)
- moved D79 356.0 mm to (404.1, 184.8)
- moved D80 321.0 mm to (404.1, 181.9)
- moved D81A1 286.3 mm to (404.1, 179.0)
- moved D81 268.6 mm to (404.1, 176.2)
- moved D81A2 258.9 mm to (404.3, 190.9)
- moved D82 219.0 mm to (404.3, 202.0)
- moved D83 164.1 mm to (404.3, 198.3)
- moved D86 154.0 mm to (404.3, 213.0)
- moved D84 147.3 mm to (404.3, 194.6)
- moved D87 147.0 mm to (404.3, 209.3)
- moved D88 136.9 mm to (404.3, 205.6)
Connections:
- D78 pad 2: Net-(D78-Pad2) -> Net-(D87-Pad2)
- D79 pad 2: Net-(D79-Pad2) -> Net-(D87-Pad2)
- D81A1 pad 2: Net-(D81A1-Pad2) -> Net-(D87-Pad2)
Routing:
- net Net-(D78-Pad2): track 146.8 -> 364.9 mm
- net Net-(D77-Pad2): track 205.5 -> 0.00 mm
- net Net-(D88-Pad2): track 225.8 -> 20.6 mm
- net Net-(D79-Pad2): track 140.6 -> 343.1 mm
- net Net-(D80-Pad2): track 140.7 -> 321.2 mm
- net Net-(D85-Pad2): track 168.3 -> 0.00 mm
- net Net-(D87-Pad2): track 195.8 -> 41.2 mm
- net Net-(D81A1-Pad2): track 141.1 -> 290.7 mm
- net Net-(D81-Pad2): track 147.1 -> 254.5 mm
- net Net-(D86-Pad2): track 165.3 -> 61.7 mm
- net Net-(D84-Pad2): track 175.6 -> 118.5 mm
- net Net-(D83-Pad2): track 195.5 -> 140.4 mm
- net row6: track 363.3 -> 400.2 mm
- net Net-(D81A2-Pad2): track 174.3 -> 194.6 mm
- net Net-(D82-Pad2): track 148.7 -> 165.1 mm
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Other:
- board size 347 x 156.3 mm -> 383.2 x 156.3 mm

Commit message: change controller; screw things up
Parts:
- removed D0, D1, D10, D11, D12, D13, D14, D15, D2, D3, D4, D5, D6, D7, D8, D9: D, Diode_THT:D_DO-35_SOD27_P7.62mm_Horizontal
- removed D89: 1n4002, Diode_THT:D_DO-35_SOD27_P7.62mm_Horizontal
- removed K_0, K_1, K_10, K_11, K_12, K_13, K_14, K_15, K_2, K_3, K_4, K_5, K_6, K_7, K_8, K_9: KEYSW, MX_Only:MXOnly-1U-NoLED
- removed RESISTOR0, RESISTOR1: 5.1k, Resistor_THT:R_Axial_DIN0207_L6.3mm_D2.5mm_P7.62mm_Horizontal
- removed USB1: HRO-TYPE-C-31-M-12, josh-connectors:USB_C_TYPE-C-31-M-14
- RPI0: footprint EM_Extras:RPi_Pico_SMD_TH -> MCU_RaspberryPi_and_Boards:RPi_Pico_SMD_TH
Connections:
- D63 pad 2: Net-(D63-Pad2) -> Net-(D63-A)
- D78 pad 2: Net-(D87-Pad2) -> Net-(D78-A)
- D79 pad 2: Net-(D87-Pad2) -> Net-(D79-A)
- D81A1 pad 2: Net-(D87-Pad2) -> Net-(D81A1-A)
- D87 pad 2: Net-(D87-Pad2) -> Net-(D87-A)
- K_63B1 pad 2: Net-(D63-Pad2) -> Net-(D63-A)
- K_78 pad 2: Net-(D78-Pad2) -> Net-(D78-A)
- K_79 pad 2: Net-(D79-Pad2) -> Net-(D79-A)
- K_81A1 pad 2: Net-(D81A1-Pad2) -> Net-(D81A1-A)
- K_87 pad 2: Net-(D87-Pad2) -> Net-(D87-A)
Routing:
- net Net-(D78-Pad2): track 364.9 -> 0.00 mm
- net Net-(D78-A): track 0.00 -> 364.9 mm
- net Net-(D79-Pad2): track 343.1 -> 0.00 mm
- net Net-(D79-A): track 0.00 -> 343.1 mm
- net Net-(D81A1-Pad2): track 290.7 -> 0.00 mm
- net Net-(D81A1-A): track 0.00 -> 290.7 mm
- net USB2_P: track 52.4 -> 0.00 mm
- net USB2_N: track 52.2 -> 0.00 mm
- net Net-(D9-Pad2): track 45.4 -> 0.00 mm
- net Net-(D87-Pad2): track 41.2 -> 0.00 mm
- net Net-(D87-A): track 0.00 -> 41.2 mm
- net Net-(D10-Pad2): track 37.9 -> 0.00 mm
- net (no net): track 0.00 -> 37.9 mm
- net Net-(D11-Pad2): track 33.3 -> 0.00 mm
- net USBVBUS: track 32.9 -> 0.00 mm, vias 2 -> 0
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