File: KiCad Files/MainPCB/ENV_KB.kicad_pcb (KiCad board)
At the start: 2 copper layers, 383.2 x 156.3 mm, 192 parts

Commit message: playing with layout
Parts:
- removed D29BS2, D62, D65, D81A1, D81A2: D, Diode_THT:D_DO-35_SOD27_P7.62mm_Horizontal
- removed I2CHeader0: Conn_01x04, Connector_PinSocket_2.54mm:PinSocket_1x04_P2.54mm_Vertical
- removed K_29BS1, K_29BS2, K_62, K_65, K_81A1, K_81A2: KEYSW, MX_Only:MXOnly-1U-NoLED
- removed K_50A1, K_64: KEYSW, MX_Only:MXOnly-1.25U-NoLED
- removed K_63: MX-NoLED, MX_Only:MXOnly-1U-NoLED
- removed STAB1: Stabilizer, Mounting_Keyboard_Stabilizer:Stabilizer_Cherry_MX_2u
- RPI0: moved to B.Cu
- moved RPI0 137.0 mm to (403.5, 86.5), turned to 180 degrees
- moved D82 20.5 mm to (394.8, 183.9), turned to -90 degrees
- moved D86 19.4 mm to (402.5, 193.7), turned to -90 degrees
- moved D87 15.6 mm to (398.6, 194.8), turned to -90 degrees
- moved D88 13.6 mm to (394.8, 195.9), turned to -90 degrees
- moved D81 8.60 mm to (398.6, 182.8), turned to -90 degrees
- moved D79 8.10 mm to (410.2, 179.5), turned to -90 degrees
- moved D78 7.42 mm to (406.4, 180.6), turned to -90 degrees
- moved D84 6.70 mm to (410.2, 191.5), turned to -90 degrees
- moved D83 6.07 mm to (406.4, 192.6), turned to -90 degrees
- moved D80 1.64 mm to (402.5, 181.7), turned to -90 degrees
- turned K_46 to 0 degrees
Routing:
- net row6: track 400.2 -> 0.00 mm
- net row0: track 371.5 -> 0.00 mm
- net Net-(D81A1-A): track 290.7 -> 0.00 mm
- net col0: track 341.6 -> 72.3 mm
- net col1: track 305.6 -> 78.0 mm
- net col2: track 275.1 -> 64.4 mm
- net col5: track 260.7 -> 65.5 mm
- net col3: track 282.1 -> 87.6 mm
- net Net-(D81A2-A): track 194.6 -> 0.00 mm
- net col4: track 245.7 -> 65.3 mm
- net col15: track 179.5 -> 0.00 mm
- net col7: track 242.7 -> 63.5 mm
- net col6: track 231.0 -> 83.7 mm
- net col14: track 197.0 -> 52.4 mm
- net Net-(D62-A): track 135.8 -> 0.00 mm
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- removed copper zone on F.Cu, net VSYS
