File: KiCad Files/MainPCB/ENV_KB.kicad_sch (KiCad schematic)
At the start: 211 parts

Commit message: change controller; screw things up
Parts:
- removed D0, D1, D10, D11, D12, D13, D14, D15, D2, D3, D4, D5, D6, D7, D8, D9: D, Diode_THT:D_DO-35_SOD27_P7.62mm_Horizontal, symbol Device:D_Small
- removed D89: 1n4002, Diode_THT:D_DO-35_SOD27_P7.62mm_Horizontal, symbol Device:D_Small
- removed K_0, K_1, K_10, K_11, K_12, K_13, K_14, K_15, K_2, K_3, K_4, K_5, K_6, K_7, K_8, K_9: KEYSW, MX_Only:MXOnly-1U-NoLED, symbol MX_Alps_Hybrid:MX-NoLED
- removed RESISTOR0, RESISTOR1: 5.1k, Resistor_THT:R_Axial_DIN0207_L6.3mm_D2.5mm_P7.62mm_Horizontal, symbol Device:R_Small
- removed USB1: HRO-TYPE-C-31-M-12, josh-connectors:USB_C_TYPE-C-31-M-14, symbol josh-connector:USB_C_U262-161N-4BVC11
- RPI0: footprint EM_Extras:RPi_Pico_SMD_TH -> RPi_Pico:RPi_Pico_SMD_TH
Connections:
- net GND: no longer RPI0.TP1 (GND_L)
- removed net USB2_N: RPI0.TP2 (USB_DM)
- removed net USB2_P: RPI0.TP3 (USB_DP)
- no-connect marks 2 -> 3

Commit message: playing with layout
Parts:
- removed D29BS2, D62, D65, D81A1, D81A2: D, Diode_THT:D_DO-35_SOD27_P7.62mm_Horizontal, symbol Device:D_Small
- removed I2CHeader0: Conn_01x04, Connector_PinSocket_2.54mm:PinSocket_1x04_P2.54mm_Vertical, symbol Connector_Generic:Conn_01x04
- removed K_29BS1, K_29BS2, K_62, K_65, K_81A1, K_81A2: KEYSW, MX_Only:MXOnly-1U-NoLED, symbol MX_Alps_Hybrid:MX-NoLED
- removed K_63: MX-NoLED, MX_only:MXOnly-ISO-ROTATED-ReversedStabilizers-NoLED, symbol MX_Alps_Hybrid:MX-NoLED
- removed K_64: KEYSW, MX_Only:MXOnly-1.25U-NoLED, symbol MX_Alps_Hybrid:MX-NoLED
